File: KiCAD-Project/Interfaces.sch (KiCad schematic (older format))
At the start: 38 parts, among them J201 XT30, J202 XT30, J203 TLE2, J204 CAN, J205 CAN, U201 TI_TCAN337G, U202 TLE5012B_E1000

Commit message: Schamtic package assigned
Package assigned, added two 100nF C's for temp sensors
Parts:
- C201, C202, C203, C204, C205, C206, C207, C208, C209, C210, C211, C212, C213, C214, C215, C216, C217, C218, C219, C220: footprint (none) -> Capacitor_SMD:C_1206_3216Metric
- C221, C222: footprint (none) -> Capacitor_SMD:C_0603_1608Metric
- J201, J202: footprint (none) -> Connector_AMASS:AMASS_XT30PW-M_1x02_P2.50mm_Horizontal
- J203: footprint (none) -> Connector_JST:JST_XH_B8B-XH-A_1x08_P2.50mm_Vertical
- J204, J205: footprint (none) -> Connector_JST:JST_XH_S3B-XH-A_1x03_P2.50mm_Horizontal
- R201, R202, R203: footprint (none) -> Resistor_SMD:R_0603_1608Metric
- TP201, TP202, TP203, TP204, TP205, TP206: footprint (none) -> TestPoint:TestPoint_Pad_D2.0mm
- U201: footprint (none) -> Package_SO:SOIC-8_3.9x4.9mm_P1.27mm
- U202: footprint Infineon-TLE5012B_E1000-* -> digikey-footprints:SOIC-8_W3.9mm
Changed lines of the file:
@@
 F 0 "J201" H 6780 1842 50  0000 L CNN
 F 1 "XT30" H 6780 1751 50  0000 L CNN
-F 2 "" H 6700 1850 50  0001 C CNN
+F 2 "Connector_AMASS:AMASS_XT30PW-M_1x02_P2.50mm_Horizontal" H 6700 1850 50  0001 C CNN
 F 3 "~" H 6700 1850 50  0001 C CNN
 	1    6700 1850
@@
 F 0 "J202" H 6780 2142 50  0000 L CNN
 F 1 "XT30" H 6780 2051 50  0000 L CNN
-F 2 "" H 6700 2150 50  0001 C CNN
+F 2 "Connector_AMASS:AMASS_XT30PW-M_1x02_P2.50mm_Horizontal" H 6700 2150 50  0001 C CNN
 F 3 "~" H 6700 2150 50  0001 C CNN
 	1    6700 2150
@@
 F 0 "J204" H 12730 2292 50  0000 L CNN
 F 1 "CAN" H 12730 2201 50  0000 L CNN
-F 2 "" H 12650 2250 50  0001 C CNN
+F 2 "Connector_JST:JST_XH_S3B-XH-A_1x03_P2.50mm_Horizontal" H 12650 2250 50  0001 C CNN
 F 3 "~" H 12650 2250 50  0001 C CNN
 	1    12650 2250
@@
 F 0 "J205" H 12730 2842 50  0000 L CNN
 F 1 "CAN" H 12730 2751 50  0000 L CNN
-F 2 "" H 12650 2800 50  0001 C CNN
+F 2 "Connector_JST:JST_XH_S3B-XH-A_1x03_P2.50mm_Horizontal" H 12650 2800 50  0001 C CNN
 F 3 "~" H 12650 2800 50  0001 C CNN
 	1    12650 2800
@@
 F 0 "J203" H 12230 6042 50  0000 L CNN
 F 1 "TLE2" H 12230 5951 50  0000 L CNN
-F 2 "" H 12150 6050 50  0001 C CNN
+F 2 "Connector_JST:JST_XH_B8B-XH-A_1x08_P2.50mm_Vertical" H 12150 6050 50  0001 C CNN
 F 3 "~" H 12150 6050 50  0001 C CNN
 	1    12150 6050
@@
 F 0 "U202" H 11900 4915 50  0000 C CNN
 F 1 "TLE5012B_E1000" H 11900 4824 50  0000 C CNN
-F 2 "Infineon-TLE5012B_E1000-*" H 11400 5050 50  0001 L CNN
+F 2 "digikey-footprints:SOIC-8_W3.9mm" H 11400 5050 50  0001 L CNN
 F 3 "http://www.infineon.com/dgdl/TLE5012B_FDS_Rev1+1.pdf?folderId=db3a30431ce5fb52011d3dd6e8012582&fileId=db3a304334fac4c601350f31c43c433f" H 11400 5150 50  0001 L CNN
 F 4 "Manufacturer URL" H 11400 5250 50  0001 L CNN "Component Link 1 Description"
@@
 F 0 "U201" H 10800 3367 50  0000 C CNN
 F 1 "TI_TCAN337G" H 10800 3276 50  0000 C CNN
-F 2 "" H 11400 2350 50  0001 C CIN
+F 2 "Package_SO:SOIC-8_3.9x4.9mm_P1.27mm" H 11400 2350 50  0001 C CIN
 F 3 "http://www.ti.com/lit/ds/symlink/tcan337.pdf" H 10800 2900 50  0001 C CNN
 	1    10800 2900
@@
 F 0 "R203" H 10059 2546 50  0000 L CNN
 F 1 "10k" H 10059 2455 50  0000 L CNN
-F 2 "" H 10000 2500 50  0001 C CNN
+F 2 "Resistor_SMD:R_0603_1608Metric" H 10000 2500 50  0001 C CNN
 F 3 "~" H 10000 2500 50  0001 C CNN
 	1    10000 2500
@@
 F 0 "C222" H 12308 4996 50  0000 R CNN
 F 1 "100n" H 12308 4905 50  0000 R CNN
-F 2 "" H 12400 4950 50  0001 C CNN
+F 2 "Capacitor_SMD:C_0603_1608Metric" H 12400 4950 50  0001 C CNN
 F 3 "~" H 12400 4950 50  0001 C CNN
 	1    12400 4950
@@
 F 0 "C221" H 11492 3196 50  0000 L CNN
 F 1 "100n" H 11492 3105 50  0000 L CNN
-F 2 "" H 11400 3150 50  0001 C CNN
+F 2 "Capacitor_SMD:C_0603_1608Metric" H 11400 3150 50  0001 C CNN
 F 3 "~" H 11400 3150 50  0001 C CNN
 	1    11400 3150
@@
 F 0 "R202" H 6509 3696 50  0000 L CNN
 F 1 "3k" H 6509 3605 50  0000 L CNN
-F 2 "" H 6450 3650 50  0001 C CNN
+F 2 "Resistor_SMD:R_0603_1608Metric" H 6450 3650 50  0001 C CNN
 F 3 "~" H 6450 3650 50  0001 C CNN
 	1    6450 3650
@@
 F 0 "R201" H 6391 3204 50  0000 R CNN
 F 1 "56k" H 6391 3295 50  0000 R CNN
-F 2 "" H 6450 3250 50  0001 C CNN
+F 2 "Resistor_SMD:R_0603_1608Metric" H 6450 3250 50  0001 C CNN
 F 3 "~" H 6450 3250 50  0001 C CNN
 	1    6450 3250
@@
 F 0 "C201" H 1592 1296 50  0000 L CNN
 F 1 "10u" H 1592 1205 50  0000 L CNN
-F 2 "" H 1500 1250 50  0001 C CNN
+F 2 "Capacitor_SMD:C_1206_3216Metric" H 1500 1250 50  0001 C CNN
 F 3 "~" H 1500 1250 50  0001 C CNN
 	1    1500 1250
@@
 F 0 "C203" H 1942 1296 50  0000 L CNN
 F 1 "10u" H 1942 1205 50  0000 L CNN
-F 2 "" H 1850 1250 50  0001 C CNN
+F 2 "Capacitor_SMD:C_1206_3216Metric" H 1850 1250 50  0001 C CNN
 F 3 "~" H 1850 1250 50  0001 C CNN
 	1    1850 1250
@@
 F 0 "C205" H 2292 1296 50  0000 L CNN
 F 1 "10u" H 2292 1205 50  0000 L CNN
-F 2 "" H 2200 1250 50  0001 C CNN
+F 2 "Capacitor_SMD:C_1206_3216Metric" H 2200 1250 50  0001 C CNN
 F 3 "~" H 2200 1250 50  0001 C CNN
 	1    2200 1250
@@
 F 0 "C207" H 2642 1296 50  0000 L CNN
 F 1 "10u" H 2642 1205 50  0000 L CNN
-F 2 "" H 2550 1250 50  0001 C CNN
+F 2 "Capacitor_SMD:C_1206_3216Metric" H 2550 1250 50  0001 C CNN
 F 3 "~" H 2550 1250 50  0001 C CNN
 	1    2550 1250
@@
 F 0 "C209" H 2992 1296 50  0000 L CNN
 F 1 "10u" H 2992 1205 50  0000 L CNN
-F 2 "" H 2900 1250 50  0001 C CNN
+F 2 "Capacitor_SMD:C_1206_3216Metric" H 2900 1250 50  0001 C CNN
 F 3 "~" H 2900 1250 50  0001 C CNN
 	1    2900 1250
@@
 F 0 "C211" H 3342 1296 50  0000 L CNN
 F 1 "10u" H 3342 1205 50  0000 L CNN
-F 2 "" H 3250 1250 50  0001 C CNN
+F 2 "Capacitor_SMD:C_1206_3216Metric" H 3250 1250 50  0001 C CNN
 F 3 "~" H 3250 1250 50  0001 C CNN
 	1    3250 1250
@@
 F 0 "C213" H 3692 1296 50  0000 L CNN
 F 1 "10u" H 3692 1205 50  0000 L CNN
-F 2 "" H 3600 1250 50  0001 C CNN
+F 2 "Capacitor_SMD:C_1206_3216Metric" H 3600 1250 50  0001 C CNN
 F 3 "~" H 3600 1250 50  0001 C CNN
 	1    3600 1250
@@
 F 0 "C215" H 4042 1296 50  0000 L CNN
 F 1 "10u" H 4042 1205 50  0000 L CNN
-F 2 "" H 3950 1250 50  0001 C CNN
+F 2 "Capacitor_SMD:C_1206_3216Metric" H 3950 1250 50  0001 C CNN
 F 3 "~" H 3950 1250 50  0001 C CNN
 	1    3950 1250
@@
 F 0 "C217" H 4392 1296 50  0000 L CNN
 F 1 "10u" H 4392 1205 50  0000 L CNN
-F 2 "" H 4300 1250 50  0001 C CNN
+F 2 "Capacitor_SMD:C_1206_3216Metric" H 4300 1250 50  0001 C CNN
 F 3 "~" H 4300 1250 50  0001 C CNN
 	1    4300 1250
@@
 F 0 "C219" H 4742 1296 50  0000 L CNN
 F 1 "10u" H 4742 1205 50  0000 L CNN
-F 2 "" H 4650 1250 50  0001 C CNN
+F 2 "Capacitor_SMD:C_1206_3216Metric" H 4650 1250 50  0001 C CNN
 F 3 "~" H 4650 1250 50  0001 C CNN
 	1    4650 1250
@@
 F 0 "C202" H 1592 2446 50  0000 L CNN
 F 1 "10u" H 1592 2355 50  0000 L CNN
-F 2 "" H 1500 2400 50  0001 C CNN
+F 2 "Capacitor_SMD:C_1206_3216Metric" H 1500 2400 50  0001 C CNN
 F 3 "~" H 1500 2400 50  0001 C CNN
 	1    1500 2400
@@
 F 0 "C204" H 1942 2446 50  0000 L CNN
 F 1 "10u" H 1942 2355 50  0000 L CNN
-F 2 "" H 1850 2400 50  0001 C CNN
+F 2 "Capacitor_SMD:C_1206_3216Metric" H 1850 2400 50  0001 C CNN
 F 3 "~" H 1850 2400 50  0001 C CNN
 	1    1850 2400
@@
 F 0 "C206" H 2292 2446 50  0000 L CNN
 F 1 "10u" H 2292 2355 50  0000 L CNN
-F 2 "" H 2200 2400 50  0001 C CNN
+F 2 "Capacitor_SMD:C_1206_3216Metric" H 2200 2400 50  0001 C CNN
 F 3 "~" H 2200 2400 50  0001 C CNN
 	1    2200 2400
@@
 F 0 "C208" H 2642 2446 50  0000 L CNN
 F 1 "10u" H 2642 2355 50  0000 L CNN
-F 2 "" H 2550 2400 50  0001 C CNN
+F 2 "Capacitor_SMD:C_1206_3216Metric" H 2550 2400 50  0001 C CNN
 F 3 "~" H 2550 2400 50  0001 C CNN
 	1    2550 2400
@@
 F 0 "C210" H 2992 2446 50  0000 L CNN
 F 1 "10u" H 2992 2355 50  0000 L CNN
-F 2 "" H 2900 2400 50  0001 C CNN
+F 2 "Capacitor_SMD:C_1206_3216Metric" H 2900 2400 50  0001 C CNN
 F 3 "~" H 2900 2400 50  0001 C CNN
 	1    2900 2400
@@
 F 0 "C212" H 3342 2446 50  0000 L CNN
 F 1 "10u" H 3342 2355 50  0000 L CNN
-F 2 "" H 3250 2400 50  0001 C CNN
+F 2 "Capacitor_SMD:C_1206_3216Metric" H 3250 2400 50  0001 C CNN
 F 3 "~" H 3250 2400 50  0001 C CNN
 	1    3250 2400
@@
 F 0 "C214" H 3692 2446 50  0000 L CNN
 F 1 "10u" H 3692 2355 50  0000 L CNN
-F 2 "" H 3600 2400 50  0001 C CNN
+F 2 "Capacitor_SMD:C_1206_3216Metric" H 3600 2400 50  0001 C CNN
 F 3 "~" H 3600 2400 50  0001 C CNN
 	1    3600 2400
@@
 F 0 "C216" H 4042 2446 50  0000 L CNN
 F 1 "10u" H 4042 2355 50  0000 L CNN
-F 2 "" H 3950 2400 50  0001 C CNN
+F 2 "Capacitor_SMD:C_1206_3216Metric" H 3950 2400 50  0001 C CNN
 F 3 "~" H 3950 2400 50  0001 C CNN
 	1    3950 2400
@@
 F 0 "C218" H 4392 2446 50  0000 L CNN
 F 1 "10u" H 4392 2355 50  0000 L CNN
-F 2 "" H 4300 2400 50  0001 C CNN
+F 2 "Capacitor_SMD:C_1206_3216Metric" H 4300 2400 50  0001 C CNN
 F 3 "~" H 4300 2400 50  0001 C CNN
 	1    4300 2400
@@
 F 0 "C220" H 4742 2446 50  0000 L CNN
 F 1 "10u" H 4742 2355 50  0000 L CNN
-F 2 "" H 4650 2400 50  0001 C CNN
+F 2 "Capacitor_SMD:C_1206_3216Metric" H 4650 2400 50  0001 C CNN
 F 3 "~" H 4650 2400 50  0001 C CNN
 	1    4650 2400
@@
 F 0 "TP206" H 11458 5518 50  0000 L CNN
 F 1 "TLE_SCK" H 11458 5427 50  0000 L CNN
-F 2 "" H 11600 5400 50  0001 C CNN
+F 2 "TestPoint:TestPoint_Pad_D2.0mm" H 11600 5400 50  0001 C CNN
 F 3 "~" H 11600 5400 50  0001 C CNN
 	1    11400 5400
@@
 F 0 "TP205" H 11058 5518 50  0000 L CNN
 F 1 "TLE_DATA" H 11058 5427 50  0000 L CNN
-F 2 "" H 11200 5400 50  0001 C CNN
+F 2 "TestPoint:TestPoint_Pad_D2.0mm" H 11200 5400 50  0001 C CNN
 F 3 "~" H 11200 5400 50  0001 C CNN
 	1    11000 5400
@@
 F 0 "TP204" H 10608 5518 50  0000 L CNN
 F 1 "TLE_CSQ" H 10608 5427 50  0000 L CNN
-F 2 "" H 10750 5400 50  0001 C CNN
+F 2 "TestPoint:TestPoint_Pad_D2.0mm" H 10750 5400 50  0001 C CNN
 F 3 "~" H 10750 5400 50  0001 C CNN
 	1    10550 5400
@@
 F 0 "TP203" H 10258 3468 50  0000 L CNN
 F 1 "CAN_RX" H 10258 3377 50  0000 L CNN
-F 2 "" H 10400 3350 50  0001 C CNN
+F 2 "TestPoint:TestPoint_Pad_D2.0mm" H 10400 3350 50  0001 C CNN
 F 3 "~" H 10400 3350 50  0001 C CNN
 	1    10200 3350
@@
 F 0 "TP202" H 9858 3468 50  0000 L CNN
 F 1 "CAN_TX" H 9858 3377 50  0000 L CNN
-F 2 "" H 10000 3350 50  0001 C CNN
+F 2 "TestPoint:TestPoint_Pad_D2.0mm" H 10000 3350 50  0001 C CNN
 F 3 "~" H 10000 3350 50  0001 C CNN
 	1    9800 3350
@@
 F 0 "TP201" H 4708 1068 50  0000 L CNN
 F 1 "V_BUS" H 4708 977 50  0000 L CNN
-F 2 "" H 4850 950 50  0001 C CNN
+F 2 "TestPoint:TestPoint_Pad_D2.0mm" H 4850 950 50  0001 C CNN
 F 3 "~" H 4850 950 50  0001 C CNN
 	1    4650 950

Commit message: pcb draft
Parts:
- removed TP201: V_BUS, TestPoint:TestPoint_Pad_D2.0mm, symbol Connector:TestPoint
- added C223, C224: 470u, Capacitor_SMD:CP_Elec_16x17.5, symbol Device:CP_Small
- added C225, C226: 1u, Capacitor_SMD:C_0603_1608Metric, symbol Device:C_Small
- added C227, C228, C229, C230, C231, C232, C233, C234, C235, C236, C237: 10u, Capacitor_SMD:C_1206_3216Metric, symbol Device:C_Small
- added F201: Polyfuse_Small, Resistor_SMD:R_1206_3216Metric, symbol Device:Polyfuse_Small
- added L201: 33u, Inductor_SMD:L_1210_3225Metric, symbol Device:L_Small
- added R204: [0R], Resistor_SMD:R_0603_1608Metric, symbol Device:R_Small
- added R205: 0R, Resistor_SMD:R_0603_1608Metric, symbol Device:R_Small
- added U203: MAX15062A, Package_DFN_QFN:DFN-8_2x2mm_P0.5mm, symbol Regulator_Switching:MAX15062A
Connections:
- net +3V3: now also C227.1, L201.2, U203.4 (FB/Vout)
- net GND: now also J201.1 (Pin_1), J202.1 (Pin_1), C223.2, C224.2, C225.2, C226.2, C227.2, C228.2, C229.2, C230.2, C231.2, C232.2, C233.2, C234.2, C235.2, C236.2, C237.2, R204.2, U203.7 (GND); no longer J201.2 (Pin_2), J202.2 (Pin_2)
- net VBUS: now also J201.2 (Pin_2), J202.2 (Pin_2), C223.1, C224.1, C228.1, C229.1, C230.1, C231.1, C232.1, C233.1, C234.1, C235.1, C236.1, C237.1, F201.2; no longer J201.1 (Pin_1), J202.1 (Pin_1), R201.2
- new net: C225.1, F201.1, R201.2, U203.1 (VIN), U203.2 (EN/UVLO)
- new net: C226.1, U203.3 (VCC)
- new net: R204.1, U203.5 (MODE)
- new net: R205.1, U203.6 (~RESET)
- new net: L201.1, U203.8 (LX)
- new net RESET: R205.2
Other:
- moved on the sheet: R201, R202
