File: KiCAD-Project/OpenTurn.sch (KiCad schematic (older format))
At the start: 128 parts, among them J1 TLE2, J2 XT30, J3 XT30, J4 JTAG/SW, J5 CAN, J6 CAN, J7 DEBUG, Q1 IAUC120N06S5N017ATMA1, Q2 IAUC120N06S5N017ATMA1, Q3 IAUC120N06S5N017ATMA1, Q4 IAUC120N06S5N017ATMA1, Q5 IAUC120N06S5N017ATMA1, Q6 IAUC120N06S5N017ATMA1, U1 TLE5012B_E1000, U2 MAX15062A, U3 TI_TCAN337G, U4 DRV8323SRTAR, U5 CY8C6244AZI-S4D92, U6 MCP9700AT-HTT, Y1 32MHz

Commit message: schematic update
schematic to multiple pages, GPIO assignment optimized for routing
Parts:
- removed C1, C39, C40, C44, C45, C46, C49, C6, C8: 0.1uF, symbol Device:C
- removed C13, C14: TBD, symbol Device:C
- removed C15, C54, C55: 100nF, symbol Device:C_Small
- removed C2, C3, C37, C38, C4, C41, C42, C9: 1uF, symbol Device:C
- removed C21, C22, C23, C24, C25, C26, C27, C28, C29, C30, C31, C32, C33, C34, C35, C36, C43, C47: 10uF, symbol Device:C
- removed C48: 4.7uF, symbol Device:C
- removed C5: 47nF, symbol Device:C
- removed C7: 10uF, Capacitor_SMD:C_1206_3216Metric, symbol Device:C
- removed C? (x9): 47pF, symbol Device:C_Small
- removed C? (x3): DNP, symbol Device:C_Small
- removed D1, D2, D3: LED, symbol Device:LED
- removed J1: TLE2, symbol Connector_Generic:Conn_01x08
- removed J2, J3: XT30, symbol Connector_Generic:Conn_01x02
- removed J4: JTAG/SW, symbol Connector_Generic:Conn_02x05_Odd_Even
- removed J5, J6: CAN, symbol Connector_Generic:Conn_01x03
- removed J7: DEBUG, symbol Connector:Conn_01x08_Male
- removed L1: 33uH, symbol Device:L
- removed L2, L3: 1k, symbol Device:L_Core_Ferrite
- removed Q1, Q2, Q3, Q4, Q5, Q6: IAUC120N06S5N017ATMA1, Package_TO_SOT_SMD:TDSON-8-1, symbol Transistor_FET:BSC028N06LS3
- removed R13, R14, R15, R5: 0R, symbol Device:R_Small
- removed R16, R8, R? (x3): 10k, symbol Device:R_Small
- removed R17, R18, R4: 4.7k, symbol Device:R
- removed R19: 56k, symbol Device:R_Small
- removed R20, R6, R7, R? (x4): 3k, symbol Device:R_Small
- removed R? (x3): 0.05m, symbol Device:R_Small
- removed TP1: MU, symbol Connector:TestPoint
- removed TP10: CAN_TX, symbol Connector:TestPoint
- removed TP11: 3v3, symbol Connector:TestPoint
- removed TP13, TP17, TP19, TP20, TP24: GND, symbol Connector:TestPoint
- removed TP14: MW, symbol Connector:TestPoint
- removed TP15: TLE_CSQ, symbol Connector:TestPoint
- removed TP16: MISO, symbol Connector:TestPoint
- removed TP2: TLE_SCK, symbol Connector:TestPoint
- removed TP21: DRV_CS, symbol Connector:TestPoint
- removed TP22: TLE1_CS, symbol Connector:TestPoint
- removed TP23: TLE2_CS, symbol Connector:TestPoint
- removed TP3: SPI_SCK, symbol Connector:TestPoint
- removed TP4: CAN_RX, symbol Connector:TestPoint
- removed TP5: VM, symbol Connector:TestPoint
- removed TP7: MV, symbol Connector:TestPoint
- removed TP8: TLE_DATA, symbol Connector:TestPoint
- removed TP9: MOSI, symbol Connector:TestPoint
- removed U1: TLE5012B_E1000, Infineon-TLE5012B_E1000-*, symbol eec:TLE5012B_E1000
- removed U2: MAX15062A, Package_DFN_QFN:DFN-8_2x2mm_P0.5mm, symbol Regulator_Switching:MAX15062A
- removed U3: TI_TCAN337G, symbol TCAN337G:TI_TCAN337G
- removed U4: DRV8323SRTAR, Package_DFN_QFN:VQFN-48-1EP_7x7mm_P0.5mm_EP5.15x5.15mm_ThermalVias, symbol DRV8323SRTAR:DRV8323SRTAR
- removed U5: CY8C6244AZI-S4D92, symbol cy8c6244azi-s4d92:CY8C6244AZI-S4D92
- removed U6: MCP9700AT-HTT, Package_TO_SOT_SMD:SOT-23, symbol Sensor_Temperature:MCP9700AT-HTT
- removed Y1: 32MHz, symbol Device:Crystal
- renumbered H1 to H101, H2 to H102, H3 to H103
Connections:
- net labels removed: +3.3V, +3V3, +48V, BUS_VOLTAGE, CAL, CANFD_RX, CANFD_TX, CAN_FAULT, CAN_H, CAN_L, CAN_RX, CAN_TX, DB_UART_RX, DB_UART_TX, DRV_CS, DRV_SCK, ENABLE, GBL, GHA, GHB, GHC, GLA, GLB, GLC, GPIO1, GPIO2, I_SENSE_A, I_SENSE_B, I_SENSE_C, MISO, MOSI, MU, MV, MW, PWM1A_H, PWM1A_L, PWM1B_H, PWM1B_L, PWM1C_H, PWM1C_L, QUAD1_A, QUAD1_B, QUAD1_I, QUAD2_A, QUAD2_B, QUAD2_I, RESET, SCL, SDA, SHA, SHB, SHC, SNA, SNB, SNC, SOA, SOB, SOC, SPA, SPB, SPC, SPI_SCK, SSC_CLK, SSC_DI, SSC_DO, STATUS_LED1, STATUS_LED2, SWDCK, SWDIO, TEMP_SYS, TLE1_CS, TLE2_CS, TLE_CSQ, TLE_DATA, VBACKUP, VCCD, VDDA, VDDD, VDDIO0, VDDIO1, VDDIO2, VDRAIN, nFAULT
- wire segments 205 -> 30
Other:
- note removed: "BOARD I/O"
- note removed: "BUCK CONVERTER"
- note removed: "BULK CAPACITANCE"
- note removed: "CAN"
- note removed: "CAN FD TRANSCIEVER"
- note removed: "CLOSE TO DRV8323"
- note removed: "CLOSE TO MCP9700"
- note removed: "DECOUPLING CAPS"
- note removed: "DRV8323"
- note removed: "GATE DRIVER"
- note removed: "HALF BRIDGES"
- note removed: "MICROCONTROLLER"
- note removed: "MISC"
- note removed: "MOTOR"
- note removed: "POSITION SENSOR"
- note removed: "TLE5012B"
- note removed: "VOLTAGE"
- note removed: "VOLTAGE DIVIDER"
- moved on the sheet: H101, H102, H103

Commit message: Schamtic package assigned
Package assigned, added two 100nF C's for temp sensors
Parts:
- H101, H102, H103: footprint (none) -> MountingHole:MountingHole_3.2mm_M3_DIN965_Pad
Changed lines of the file:
@@
 F 0 "H101" H 1250 5499 50  0000 L CNN
 F 1 "3.2mm" H 1250 5408 50  0000 L CNN
-F 2 "" H 1150 5450 50  0001 C CNN
+F 2 "MountingHole:MountingHole_3.2mm_M3_DIN965_Pad" H 1150 5450 50  0001 C CNN
 F 3 "~" H 1150 5450 50  0001 C CNN
 	1    1150 5450
@@
 F 0 "H102" H 1250 5999 50  0000 L CNN
 F 1 "3.2mm" H 1250 5908 50  0000 L CNN
-F 2 "" H 1150 5950 50  0001 C CNN
+F 2 "MountingHole:MountingHole_3.2mm_M3_DIN965_Pad" H 1150 5950 50  0001 C CNN
 F 3 "~" H 1150 5950 50  0001 C CNN
 	1    1150 5950
@@
 F 0 "H103" H 1250 6499 50  0000 L CNN
 F 1 "3.2mm" H 1250 6408 50  0000 L CNN
-F 2 "" H 1150 6450 50  0001 C CNN
+F 2 "MountingHole:MountingHole_3.2mm_M3_DIN965_Pad" H 1150 6450 50  0001 C CNN
 F 3 "~" H 1150 6450 50  0001 C CNN
 	1    1150 6450

Commit message: pcb draft
Changed lines of the file:
@@
 F14 "ENCODER_DATA" I R 4000 2650 50
 F15 "V_BUS_SENSE" I R 4000 1200 50
+F16 "RESET" I R 4000 1300 50
 $EndSheet
 $Sheet
@@
 F30 "DRV_SCK" I R 8400 3700 50
 F31 "DRV_CS" I R 8400 3800 50
+F32 "RESET" I L 5000 1300 50
 $EndSheet
 Wire Wire Line
@@
 Wire Wire Line
 	8400 3800 9500 3800
+Wire Wire Line
+	4000 1300 5000 1300
 $EndSCHEMATC
